File: PCBs/DriveSystem/DriveSystem.sch (KiCad schematic (older format))
At the start: 12 parts

Commit message: added ultrasonic sensors
Parts:
- removed C?: 2.2u, symbol pspice:CAP
- removed C?: 10u, symbol pspice:CAP
- removed C?: 0.1u, symbol pspice:CAP
- added C?: 0.22u, symbol Device:C
- added C? (x2): 0.1u, symbol Device:C
- added C?: 10u, symbol Device:C
- added C?: 2.2u, symbol Device:C
- added J? (x2): Conn_01x04_Male, symbol Connector:Conn_01x04_Male
- added J?: Screw_Terminal_01x02, symbol Connector:Screw_Terminal_01x02
- added U?: LM7805_TO220, Package_TO_SOT_THT:TO-220-3_Vertical, symbol Regulator_Linear:LM7805_TO220
Connections:
- net labels added: +12V, +5V, ECHOl, ECHOr, TRIG
- wire segments 46 -> 76
Other:
- note added: "-Make sure ultrasonic pins oriented correctly"
- note added: "-Verify package on the 5V regulator\n"
