File: PCBs/DriveSystem/DriveSystem.sch (KiCad schematic (older format))
At the start: 41 parts, among them J1 Conn_01x05_Male, J10 Conn_01x04_Female, J11 Conn_01x03_Male, J2 Conn_01x14_Female, J3 Conn_01x04_Female, J4 Conn_01x03_Male, J5 Screw_Terminal_01x02, J6 Screw_Terminal_01x02, J7 Conn_01x04_Male, J8 Conn_01x04_Male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

Commit message: Started pcb tracing
Parts:
- added C13, C15, C16: .1u, Capacitor_SMD:C_0805_2012Metric_Pad1.15x1.40mm_HandSolder, symbol Device:C
- added C14: 10u, Capacitor_SMD:C_0805_2012Metric_Pad1.15x1.40mm_HandSolder, symbol Device:C
- added J12: Servo_Header, Connector_PinHeader_2.54mm:PinHeader_1x03_P2.54mm_Vertical, symbol Connector:Conn_01x03_Male
- added J13: Load_Cell_Header, Connector_PinSocket_2.54mm:PinSocket_1x04_P2.54mm_Vertical, symbol Connector:Conn_01x04_Female
- added JP1: SolderJumper_2_Bridged, Jumper:SolderJumper-2_P1.3mm_Bridged2Bar_Pad1.0x1.5mm, symbol Jumper:SolderJumper_2_Bridged
- added L1: 3.3u, Inductor_SMD:L_0805_2012Metric_Pad1.15x1.40mm_HandSolder, symbol Device:L
- added Q3: MMBT3906, Package_TO_SOT_SMD:SOT-23, symbol Transistor_BJT:MMBT3906
- added R10: 8.2k, Resistor_SMD:R_0805_2012Metric_Pad1.15x1.40mm_HandSolder, symbol Device:R
- added R11, R12: 100, Resistor_SMD:R_0805_2012Metric_Pad1.15x1.40mm_HandSolder, symbol Device:R
- added R13: 10k, Resistor_SMD:R_0805_2012Metric_Pad1.15x1.40mm_HandSolder, symbol Device:R
- added R9: 20k, Resistor_SMD:R_0805_2012Metric_Pad1.15x1.40mm_HandSolder, symbol Device:R
- added U5: HX711, Package_SO:SOP-16_4.55x10.3mm_P1.27mm, symbol LoadCell:HX711
- J1: value Conn_01x05_Male -> SWD_Header; footprint Connector_PinHeader_2.54mm:PinHeader_1x01_P2.54mm_Vertical -> Connector_PinHeader_2.54mm:PinHeader_1x05_P2.54mm_Vertical
- J10: value Conn_01x04_Female -> Stack_Light; footprint Connector_PinSocket_2.54mm:PinSocket_1x01_P2.54mm_Vertical -> Connector_PinSocket_2.54mm:PinSocket_1x04_P2.54mm_Vertical
- J11: value Conn_01x03_Male -> LPS_Header; footprint Connector_PinHeader_2.54mm:PinHeader_1x01_P2.54mm_Vertical -> Connector_PinHeader_2.54mm:PinHeader_1x03_P2.54mm_Vertical
- J2: value Conn_01x14_Female -> Touchscreen_Header; footprint Connector_PinSocket_2.54mm:PinSocket_1x01_P2.54mm_Vertical -> Connector_PinSocket_2.54mm:PinSocket_1x14_P2.54mm_Vertical
- J3: value Conn_01x04_Female -> SD_Card_Header; footprint Connector_PinSocket_2.54mm:PinSocket_1x01_P2.54mm_Vertical -> Connector_PinSocket_2.54mm:PinSocket_1x04_P2.54mm_Vertical
- J4: value Conn_01x03_Male -> Input_12V; footprint TerminalBlock_4Ucon:TerminalBlock_4Ucon_1x03_P3.50mm_Horizontal -> Connector_PinHeader_2.54mm:PinHeader_1x03_P2.54mm_Vertical
- J7: value Conn_01x04_Male -> Right_Ultrasonic; footprint Connector_PinHeader_2.54mm:PinHeader_1x01_P2.54mm_Vertical -> Connector_PinHeader_2.54mm:PinHeader_1x04_P2.54mm_Vertical
- J8: value Conn_01x04_Male -> Left_Ultrasonic; footprint Connector_PinHeader_2.54mm:PinHeader_1x01_P2.54mm_Vertical -> Connector_PinHeader_2.54mm:PinHeader_1x04_P2.54mm_Vertical
- J9: value Conn_01x06_Male -> IMU_Header; footprint Connector_PinHeader_2.54mm:PinHeader_1x01_P2.54mm_Vertical -> Connector_PinHeader_2.54mm:PinHeader_1x06_P2.54mm_Vertical
Connections:
- net +3V3: now also Q3.2 (E), R13.1, U5.1 (VSUP)
- net +5V: now also J12.2 (Pin_2), U5.16 (DVDD)
- net BIN1: now also U1.44 (PA11); no longer U1.43 (PA10)
- net BIN2: now also U1.43 (PA10); no longer U1.44 (PA11)
- net GND: now also C13.1, C14.1, C15.2, J12.1 (Pin_1), J13.2 (Pin_2), JP1.2 (B), R10.2, U5.14 (XI), U5.5 (AGND)
- net at U2.5 (BOUT2): now also J6.1 (Pin_1); no longer J6.2 (Pin_2)
- net at U2.7 (BOUT1): now also J6.2 (Pin_2); no longer J6.1 (Pin_1)
- new net: JP1.1 (A), R13.2, U5.15 (RATE)
- new net: Q3.1 (B), U5.2 (BASE)
- new net: L1.2, Q3.3 (C), R9.1, U5.3 (AVDD)
- new net: R10.1, R9.2, U5.4 (VFB)
- new net: C15.1, U5.6 (VBG)
- new net: C16.2, R11.1, U5.7 (INA-)
- new net: C16.1, R12.1, U5.8 (INA+)
- new net LC_AVDD: C13.2, C14.2, J13.1 (Pin_1), L1.1
- new net LC_DOUT: U5.12 (DOUT)
- new net LC_INA+: J13.4 (Pin_4), R12.2
- new net LC_INA-: J13.3 (Pin_3), R11.2
- new net LC_SCK: U5.11 (PD_SCK)
- new net SV_FB: J12.3 (Pin_3)
Other:
- note added: "-Check Tranny\n"
- note added: "-Determine microcontroller pins\n"
- note added: "-Determine servo pins\n"
- note added: "-Need to decide data rate"
- note added: "-Regular header?\n"
- note added: "-Switch BIN1 and BIN2 in the software\n"
- note added: "-Verify package\n"
- note added: "-Will need some decoupling caps\n"
- note added: "Load Cell Amp\n"
- note added: "Load Cell Header\n"
- note added: "Servo Header"

Commit message: First pcb thing done (gotta redo a lot of it)
Parts:
- U5: symbol LoadCell:HX711 -> DriveSystem-rescue:HX711-LoadCell
Connections:
- net Buzzer: now also Q2.2 (G1); no longer Q2.4 (G2)
- net sGreen: now also Q1.4 (G2); no longer Q1.2 (G1)
- net sGreeni: now also Q1.5 (D2), Q1.6 (D2); no longer Q1.7 (D1), Q1.8 (D1)
- net sRed: now also Q2.4 (G2); no longer Q2.2 (G1)
- net sRedi: now also Q2.5 (D2), Q2.6 (D2); no longer Q2.7 (D1), Q2.8 (D1)
- net sYellow: now also Q1.2 (G1); no longer Q1.4 (G2)
- net sYellowi: now also Q1.7 (D1), Q1.8 (D1); no longer Q1.5 (D2), Q1.6 (D2)
- new net: BZ1.2 (+), Q2.7 (D1), Q2.8 (D1)
Other:
- moved on the sheet: BZ1
Changed lines of the file:
@@
 EESchema Schematic File Version 4
 LIBS:DriveSystem-cache
-EELAYER 29 0
+EELAYER 30 0
 EELAYER END
 $Descr A3 16535 11693
@@
 Wire Wire Line
 	10850 7150 10600 7150
+Text Label 9150 7150 0    50   ~ 0
+sGreen
 Text Label 8500 7150 0    50   ~ 0
-sGreen
-Text Label 9150 7150 0    50   ~ 0
 sYellow
+Text Label 10600 7150 0    50   ~ 0
+sRed
 Text Label 9850 7150 0    50   ~ 0
-sRed
-Text Label 10600 7150 0    50   ~ 0
 Buzzer
 Text Label 1150 4200 0    50   ~ 0
@@
 	1    0    0    -1
 $EndComp
+Text Label 9400 6800 0    50   ~ 0
+sGreeni
 Text Label 8750 6800 0    50   ~ 0
-sGreeni
-Text Label 9400 6800 0    50   ~ 0
 sYellowi
-Text Label 10100 6800 0    50   ~ 0
+Text Label 10800 6800 0    50   ~ 0
 sRedi
 Text Notes 6650 1700 0    50   ~ 0
@@
 Text Notes 6650 1800 0    50   ~ 0
 -Final sd card decision\n
-Text Notes 9400 6550 0    50   ~ 0
+Text Notes 8100 6450 0    50   ~ 0
 Stack Light / Buzzer MOSFETs\n
 Text Notes 9700 8000 0    50   ~ 0
@@
 L Device:Buzzer BZ1
 U 1 1 5DD3DCBB
-P 10900 6550
-F 0 "BZ1" H 11052 6579 50  0000 L CNN
-F 1 "Buzzer" H 11052 6488 50  0000 L CNN
-F 2 "RoboPicasso:Mallory-PK-27H25PQ-Buzzer" V 10875 6650 50  0001 C CNN
-F 3 "~" V 10875 6650 50  0001 C CNN
-	1    10900 6550
-	1    0    0    -1
-$EndComp
-Wire Wire Line
-	10800 6650 10800 6800
+P 10200 6550
+F 0 "BZ1" H 10352 6579 50  0000 L CNN
+F 1 "Buzzer" H 10352 6488 50  0000 L CNN
+F 2 "RoboPicasso:Mallory-PK-27H25PQ-Buzzer" V 10175 6650 50  0001 C CNN
+F 3 "~" V 10175 6650 50  0001 C CNN
+	1    10200 6550
+	1    0    0    -1
+$EndComp
+Wire Wire Line
+	10100 6650 10100 6800
 $Comp
 L power:+12V #PWR044
 U 1 1 5DD4EA95
-P 10800 6350
-F 0 "#PWR044" H 10800 6200 50  0001 C CNN
-F 1 "+12V" H 10815 6523 50  0000 C CNN
-F 2 "" H 10800 6350 50  0001 C CNN
-F 3 "" H 10800 6350 50  0001 C CNN
-	1    10800 6350
-	1    0    0    -1
-$EndComp
-Wire Wire Line
-	10800 6350 10800 6450
+P 10100 6350
+F 0 "#PWR044" H 10100 6200 50  0001 C CNN
+F 1 "+12V" H 10115 6523 50  0000 C CNN
+F 2 "" H 10100 6350 50  0001 C CNN
+F 3 "" H 10100 6350 50  0001 C CNN
+	1    10100 6350
+	1    0    0    -1
+$EndComp
+Wire Wire Line
+	10100 6350 10100 6450
 $Comp
 L Regulator_Linear:LM2936-3.3_TO92 U4
@@
 $EndComp
 $Comp
-L LoadCell:HX711 U5
+L DriveSystem-rescue:HX711-LoadCell U5
 U 1 1 5DDA517A
 P 13800 4900

Commit message: modfied pcb
Parts:
- removed BZ1: Buzzer, RoboPicasso:Mallory-PK-27H25PQ-Buzzer, symbol Device:Buzzer
- added J14: Conn_01x02_Male, Connector_PinHeader_2.54mm:PinHeader_1x02_P2.54mm_Vertical, symbol Connector:Conn_01x02_Male
- added J15: Conn_01x07_Female, symbol Connector:Conn_01x07_Female
Connections:
- net +12V: now also J14.1 (Pin_1)
- net SV_FB: now also U1.61 (PB8)
- net PF4: now reaches U1.18 (PF4)
- net PF5: now reaches U1.19 (PF5)
- net PC13: now reaches U1.2 (PC13)
- net PC4: now reaches U1.24 (PC4)
- net PC4: now also J15.7 (Pin_7)
- net PC5: now reaches U1.25 (PC5)
- net PC5: now also J15.6 (Pin_6)
- net PB0: now reaches U1.26 (PB0)
- net PB0: now also J15.5 (Pin_5)
- net PB1: now reaches U1.27 (PB1)
- net PB1: now also J15.4 (Pin_4)
- net PB2: now reaches U1.28 (PB2)
- net PB2: now also J15.3 (Pin_3)
- net PB10: now reaches U1.29 (PB10)
- net PB10: now also J15.2 (Pin_2)
- net PC14: now reaches U1.3 (PC14)
- net PB11: now reaches U1.30 (PB11)
- net PB11: now also J15.1 (Pin_1)
- net PC15: now reaches U1.4 (PC15)
- net PC9: now reaches U1.40 (PC9)
- net PA12: now reaches U1.45 (PA12)
- net PF6: now reaches U1.47 (PF6)
- net PF7: now reaches U1.48 (PF7)
- net PF0: now reaches U1.5 (PF0)
- net PC10: now reaches U1.51 (PC10)
- net PC11: now reaches U1.52 (PC11)
- net PC12: now reaches U1.53 (PC12)
- net PD2: now reaches U1.54 (PD2)
- net PB3: now reaches U1.55 (PB3)
- net PB4: now reaches U1.56 (PB4)
- net PB5: now reaches U1.57 (PB5)
- net PF1: now reaches U1.6 (PF1)
- net Buzz: now reaches Q2.7 (D1), Q2.8 (D1)
- net Buzz: now also J14.2 (Pin_2)
Changed lines of the file:
@@
 EESchema Schematic File Version 4
 LIBS:DriveSystem-cache
-EELAYER 30 0
+EELAYER 29 0
 EELAYER END
 $Descr A3 16535 11693
@@
 3V Regulator (REPLACE)
 $Comp
-L Device:Buzzer BZ1
-U 1 1 5DD3DCBB
-P 10200 6550
-F 0 "BZ1" H 10352 6579 50  0000 L CNN
-F 1 "Buzzer" H 10352 6488 50  0000 L CNN
-F 2 "RoboPicasso:Mallory-PK-27H25PQ-Buzzer" V 10175 6650 50  0001 C CNN
-F 3 "~" V 10175 6650 50  0001 C CNN
-	1    10200 6550
-	1    0    0    -1
-$EndComp
-Wire Wire Line
-	10100 6650 10100 6800
-$Comp
-L power:+12V #PWR044
-U 1 1 5DD4EA95
-P 10100 6350
-F 0 "#PWR044" H 10100 6200 50  0001 C CNN
-F 1 "+12V" H 10115 6523 50  0000 C CNN
-F 2 "" H 10100 6350 50  0001 C CNN
-F 3 "" H 10100 6350 50  0001 C CNN
-	1    10100 6350
-	1    0    0    -1
-$EndComp
-Wire Wire Line
-	10100 6350 10100 6450
-$Comp
 L Regulator_Linear:LM2936-3.3_TO92 U4
 U 1 1 5DD687C8
@@
 Text Notes 13500 1100 0    50   ~ 0
 -Switch BIN1 and BIN2 in the software\n
+$Comp
+L Connector:Conn_01x02_Male J14
+U 1 1 5E5C774B
+P 11100 8400
+F 0 "J14" H 11208 8581 50  0000 C CNN
+F 1 "Conn_01x02_Male" H 11208 8490 50  0000 C CNN
+F 2 "Connector_PinHeader_2.54mm:PinHeader_1x02_P2.54mm_Vertical" H 11100 8400 50  0001 C CNN
+F 3 "~" H 11100 8400 50  0001 C CNN
+	1    11100 8400
+	1    0    0    -1
+$EndComp
+Wire Wire Line
+	11300 8500 11500 8500
+$Comp
+L power:+12V #PWR0101
+U 1 1 5E5F7F08
+P 11600 8350
+F 0 "#PWR0101" H 11600 8200 50  0001 C CNN
+F 1 "+12V" H 11615 8523 50  0000 C CNN
+F 2 "" H 11600 8350 50  0001 C CNN
+F 3 "" H 11600 8350 50  0001 C CNN
+	1    11600 8350
+	1    0    0    -1
+$EndComp
+Wire Wire Line
+	11600 8350 11600 8400
+Wire Wire Line
+	11300 8400 11600 8400
+Text Label 10100 6800 0    50   ~ 0
+Buzz
+Text Label 11500 8500 2    50   ~ 0
+Buzz
+Wire Wire Line
+	2750 3700 3350 3700
+Text Label 3350 3700 2    50   ~ 0
+PA12
+Text Label 3350 4200 2    50   ~ 0
+PB0
+Wire Wire Line
+	3350 4200 2750 4200
+Text Label 3350 4300 2    50   ~ 0
+PB1
+Wire Wire Line
+	3350 4300 2750 4300
+Text Label 3350 4400 2    50   ~ 0
+PB2
+Text Label 3350 4500 2    50   ~ 0
+PB3
+Text Label 3350 4600 2    50   ~ 0
+PB4
+Text Label 3350 4700 2    50   ~ 0
+PB5
+Text Label 3350 5200 2    50   ~ 0
+PB10
+Text Label 3350 5300 2    50   ~ 0
+PB11
+Text Label 1150 3300 0    50   ~ 0
+PF0
+Text Label 1150 3400 0    50   ~ 0
+PF1
+Text Label 1150 3500 0    50   ~ 0
+PF4
+Text Label 1150 3600 0    50   ~ 0
+PF5
+Text Label 1150 3700 0    50   ~ 0
+PF6
+Text Label 1150 3800 0    50   ~ 0
+PF7
+Text Label 1150 4000 0    50   ~ 0
+PD2
+Text Label 1150 4600 0    50   ~ 0
+PC4
+Text Label 1150 5100 0    50   ~ 0
+PC9
+Wire Wire Line
+	1150 5100 1550 5100
+Wire Wire Line
+	1150 4600 1550 4600
+Wire Wire Line
+	1550 3800 1150 3800
+Wire Wire Line
+	1150 4000 1550 4000
+Wire Wire Line
+	1150 3700 1550 3700
+Wire Wire Line
+	1550 3600 1150 3600
+Wire Wire Line
+	1150 3500 1550 3500
+Wire Wire Line
+	1550 3400 1150 3400
+Wire Wire Line
+	1150 3300 1550 3300
+Text Label 1150 5200 0    50   ~ 0
+PC10
+Text Label 1150 5300 0    50   ~ 0
+PC11
+Text Label 1150 5400 0    50   ~ 0
+PC12
+Text Label 1150 5500 0    50   ~ 0
+PC13
+Text Label 1150 5600 0    50   ~ 0
+PC14
+Text Label 1150 5700 0    50   ~ 0
+PC15
+Wire Wire Line
+	1150 5700 1550 5700
+Wire Wire Line
+	1550 5600 1150 5600
+Wire Wire Line
+	1150 5500 1550 5500
+Wire Wire Line
+	1550 5400 1150 5400
+Wire Wire Line
+	1150 5300 1550 5300
+Wire Wire Line
+	1550 5200 1150 5200
+Text Label 1150 4700 0    50   ~ 0
+PC5
+Wire Wire Line
+	1550 4700 1150 4700
+Wire Wire Line
+	2750 5300 3350 5300
+Wire Wire Line
+	3350 5200 2750 5200
+Wire Wire Line
+	2750 5000 3350 5000
+Wire Wire Line
+	3350 4700 2750 4700
+Wire Wire Line
+	2750 4600 3350 4600
+Wire Wire Line
+	3350 4500 2750 4500
+Wire Wire Line
+	2750 4400 3350 4400
+Wire Wire Line
+	7850 8200 8200 8200
+Wire Wire Line
+	7850 8300 8200 8300
+Wire Wire Line
+	7850 8400 8200 8400
+Wire Wire Line
+	7850 8500 8200 8500
+Wire Wire Line
+	7850 8600 8200 8600
+Text Label 8200 8200 2    50   ~ 0
+PB11
+Text Label 8200 8300 2    50   ~ 0
+PB10
+Text Label 8200 8400 2    50   ~ 0
+PB2
+Text Label 8200 8500 2    50   ~ 0
+PB1
+Text Label 8200 8600 2    50   ~ 0
+PB0
+Text Label 3350 5000 2    50   ~ 0
+SV_FB
+$Comp
+L Connector:Conn_01x07_Female J15
+U 1 1 5EC33544
+P 7650 8500
+F 0 "J15" H 7678 8526 50  0000 L CNN
+F 1 "Conn_01x07_Female" H 7678 8435 50  0000 L CNN
+F 2 "" H 7650 8500 50  0001 C CNN
+F 3 "~" H 7650 8500 50  0001 C CNN
+	1    7650 8500
+	-1   0    0    -1
+$EndComp
+Text Label 8200 8700 2    50   ~ 0
+PC5
+Text Label 8200 8800 2    50   ~ 0
+PC4
+Wire Wire Line
+	7850 8700 8200 8700
+Wire Wire Line
+	7850 8800 8200 8800
 $EndSCHEMATC
