File: PCBs/DriveSystem/DriveSystem.kicad_pcb (KiCad board)
At the start: 2 copper layers, 56 parts, among them J1 SWD_Header, J10 Stack_Light, J11 LPS_Header, J12 Servo_Header, J13 Load_Cell_Header, J2 Touchscreen_Header, J3 SD_Card_Header, J4 Input_12V, J5 Screw_Terminal_01x02, J6 Screw_Terminal_01x02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

Commit message: First pcb thing done (gotta redo a lot of it)
Parts:
- moved C6 79.0 mm to (261.9, 106.4), turned to 180 degrees
- moved C3 78.4 mm to (249.3, 106.4), turned to 180 degrees
- moved U4 77.8 mm to (245.8, 102.4)
- moved D1 73.5 mm to (241.1, 100.6), turned to 270 degrees
- moved U3 72.7 mm to (256.6, 102.9), turned to 0 degrees
- moved C2 71.2 mm to (256.2, 106.4)
- moved C7 68.1 mm to (244.8, 106.3)
- moved R2 67.6 mm to (241.1, 105.3), turned to 90 degrees
- moved C12 66.6 mm to (186.6, 103.4)
- moved J10 48.6 mm to (190.3, 107.4), turned to 90 degrees
- moved J12 43.7 mm to (223.4, 100.8), turned to 90 degrees
- moved Q2 37.3 mm to (228.4, 85.8)
- moved C8 35.3 mm to (223.4, 79.8)
- moved J9 34.3 mm to (212.3, 107.2)
- moved J4 31.5 mm to (184.5, 107.4)
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Connections:
- Q1 pad 2: /sGreen -> /sYellow
- Q1 pad 4: /sYellow -> /sGreen
- Q1 pad 5: /sYellowi -> /sGreeni
- Q1 pad 6: /sYellowi -> /sGreeni
- Q1 pad 7: /sGreeni -> /sYellowi
- Q1 pad 8: /sGreeni -> /sYellowi
- Q2 pad 2: /sRed -> /Buzzer
- Q2 pad 4: /Buzzer -> /sRed
- Q2 pad 5: Net-(BZ1-Pad2) -> /sRedi
- Q2 pad 6: Net-(BZ1-Pad2) -> /sRedi
- Q2 pad 7: /sRedi -> Net-(BZ1-Pad2)
- Q2 pad 8: /sRedi -> Net-(BZ1-Pad2)
Routing:
- net /sRedi: track 0.00 -> 55.3 mm, vias 0 -> 2
- net /sYellowi: track 0.00 -> 54.1 mm, vias 0 -> 2
- net /sGreeni: track 0.00 -> 52.1 mm, vias 0 -> 2
- net /NRST: track 0.00 -> 46.2 mm, vias 0 -> 3
- net /T_IRQ: track 0.00 -> 42.0 mm, vias 0 -> 2
- net /T_CLK: track 0.00 -> 30.3 mm, vias 0 -> 2
- net GND: track 0.00 -> 29.6 mm
- net /T_CS: track 0.00 -> 26.1 mm, vias 0 -> 2
- net /T_DO: track 0.00 -> 24.6 mm, vias 0 -> 2
- net /T_DIN: track 0.00 -> 22.0 mm
- net /LPS_SRL: track 0.00 -> 17.6 mm, vias 0 -> 2
- net /LCD_SCK: track 0.00 -> 16.1 mm, vias 0 -> 2
- net /SWDIO: track 0.00 -> 16.0 mm, vias 0 -> 2
- net /IMU_SDA: track 0.00 -> 15.8 mm, vias 0 -> 2
- net /LCD_DC: track 0.00 -> 15.6 mm, vias 0 -> 2
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- added copper zone on F.Cu, net +12V
Other:
- board text removed: "-Make sure to fix 12V traces"

Commit message: Pcb almost done
:
Parts:
- removed BZ1: Buzzer, RoboPicasso:Mallory-PK-27H25PQ-Buzzer
- removed R7: 330k, Resistor_SMD:R_0805_2012Metric_Pad1.15x1.40mm_HandSolder
- removed R8: 100k, Resistor_SMD:R_0805_2012Metric_Pad1.15x1.40mm_HandSolder
- added 1: MountingHole_5mm_Pad, MountingHole:MountingHole_5mm_Pad, F.Cu at (173.7, 66.6)
- added 2: MountingHole_5mm_Pad, MountingHole:MountingHole_5mm_Pad, F.Cu at (259.0, 66.6)
- added 3: MountingHole_5mm_Pad, MountingHole:MountingHole_5mm_Pad, F.Cu at (173.7, 113.5)
- added 4: MountingHole_5mm_Pad, MountingHole:MountingHole_5mm_Pad, F.Cu at (259.0, 113.7)
- added J14: Conn_01x02_Male, Connector_PinHeader_2.54mm:PinHeader_1x02_P2.54mm_Vertical, F.Cu at (237.7, 103.1)
- added J15: Conn_01x05_Female, Connector_PinSocket_2.54mm:PinSocket_1x05_P2.54mm_Vertical, F.Cu at (170.9, 75.1)
- moved J4 51.9 mm to (236.4, 107.5)
- moved J13 36.4 mm to (243.4, 71.6), turned to 270 degrees
- moved R12 20.9 mm to (247.2, 79.2), turned to 90 degrees
- moved R11 19.5 mm to (249.5, 79.2), turned to 90 degrees
- moved L1 19.1 mm to (259.1, 79.2), turned to 270 degrees
- moved C14 18.3 mm to (256.8, 79.2), turned to 90 degrees
- moved C13 18.0 mm to (254.5, 79.2), turned to 90 degrees
- moved C16 14.7 mm to (248.3, 83.7), turned to 0 degrees
- moved Q3 13.3 mm to (259.2, 83.7), turned to 90 degrees
- moved C15 12.5 mm to (251.5, 83.7), turned to 90 degrees
- moved R9 11.8 mm to (256.1, 83.7), turned to 90 degrees
- moved R10 11.7 mm to (253.8, 83.7), turned to 90 degrees
- moved JP1 11.4 mm to (257.8, 97.7), turned to 0 degrees
- moved R13 7.44 mm to (254.1, 97.8)
- moved J2 7.36 mm to (186.2, 71.6)
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Connections:
- net Net-(BZ1-Pad2) renamed /Buzz
- net Net-(U1-Pad18) renamed /PF4
- net Net-(U1-Pad19) renamed /PF5
- net Net-(U1-Pad2) renamed /PC13
- net Net-(U1-Pad24) renamed /PC4
- net Net-(U1-Pad25) renamed /PC5
- net Net-(U1-Pad3) renamed /PC14
- net Net-(U1-Pad4) renamed /PC15
- net Net-(U1-Pad40) renamed /PC9
- net Net-(U1-Pad45) renamed /PA12
- net Net-(U1-Pad47) renamed /PF6
- net Net-(U1-Pad48) renamed /PF7
- net Net-(U1-Pad5) renamed /PF0
- net Net-(U1-Pad51) renamed /PC10
- net Net-(U1-Pad52) renamed /PC11
- net Net-(U1-Pad53) renamed /PC12
- net Net-(U1-Pad54) renamed /PD2
- net Net-(U1-Pad55) renamed /PB3
- net Net-(U1-Pad56) renamed /PB4
- net Net-(U1-Pad57) renamed /PB5
- net Net-(U1-Pad6) renamed /PF1
- U1 pad 26: Net-(U1-Pad26) -> /PB0
- U1 pad 27: Net-(U1-Pad27) -> /PB1
- U1 pad 28: Net-(U1-Pad28) -> /PB2
- U1 pad 29: Net-(U1-Pad29) -> /PB10
- U1 pad 30: Net-(U1-Pad30) -> /PB11
- U1 pad 61: Net-(U1-Pad61) -> /SV_FB
Routing:
- net +3V3: track 9.55 -> 99.4 mm, vias 0 -> 7
- net GND: track 29.6 -> 116.0 mm, vias 0 -> 30
- net +5V: track 3.99 -> 59.3 mm, vias 0 -> 2
- net /PB11: track 0.00 -> 38.1 mm
- net /BATLVL: track 0.00 -> 37.7 mm, vias 0 -> 4
- net /ECHOr: track 3.28 -> 31.1 mm, vias 1 -> 2
- net /ECHOl: track 9.13 -> 36.8 mm, vias 1 -> 3
- net /Buzz: track 0.00 -> 26.7 mm, vias 0 -> 2
- net /TRIG: track 5.08 -> 31.8 mm, vias 0 -> 2
- net /SV_FB: track 0.00 -> 24.4 mm, vias 0 -> 1
- net /LC_AVDD: track 8.28 -> 19.7 mm
- net /LC_INA+: track 4.40 -> 14.2 mm
- net /LC_INA-: track 4.52 -> 13.9 mm
- net /LCD_DC: track 15.6 -> 24.4 mm
- net /T_IRQ: track 42.0 -> 49.5 mm
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- added copper zone on F.Cu, net +3V3
- added copper zone on B.Cu, net GND
- added copper zone on F.Cu, net Net-(J5-Pad1)
- added copper zone on F.Cu, net Net-(J5-Pad2)
- added copper zone on F.Cu, net Net-(J6-Pad1)
- added copper zone on F.Cu, net Net-(J6-Pad2)
- added copper zone on F.Cu, net Net-(R3-Pad2)
- added copper zone on F.Cu, net Net-(R4-Pad2)
Other:
- board text added: "+3V3"
- board text added: "GND"
- board text added: "LCD_CS"
- board text added: "LCD_DC"
- board text added: "LCD_MOSI"
- board text added: "LCD_RST"
- board text added: "LCD_SCK"
- board text added: "RoboPicasso ECE 49022 Designed By: Mark Miller Rev: 1"
- board text added: "T_CLK"
- board text added: "T_CS"
- board text added: "T_DIN"
- board text added: "T_DO"
- board text added: "T_IRQ"
